File: power.kicad_sch (KiCad schematic)
At the start: 39 parts, among them U1 AP63205WU, U10 AP63200WU, U9 AP63203WU

Commit message: cleanup, logical arrangement of connectors, short paths where possible and step files for all components
Parts:
- JP1: renamed from JP2; footprint TestPoint:TestPoint_2Pads_Pitch2.54mm_Drill0.8mm -> Connector_PinHeader_2.54mm:PinHeader_1x02_P2.54mm_Vertical
- JP10: renamed from JP9; footprint TestPoint:TestPoint_2Pads_Pitch2.54mm_Drill0.8mm -> Connector_PinHeader_2.54mm:PinHeader_1x02_P2.54mm_Vertical
- JP11, JP12: footprint TestPoint:TestPoint_2Pads_Pitch2.54mm_Drill0.8mm -> Connector_PinHeader_2.54mm:PinHeader_1x02_P2.54mm_Vertical
- JP2: renamed from JP5; footprint TestPoint:TestPoint_2Pads_Pitch2.54mm_Drill0.8mm -> Connector_PinHeader_2.54mm:PinHeader_1x02_P2.54mm_Vertical
- JP3: renamed from JP7; footprint TestPoint:TestPoint_2Pads_Pitch2.54mm_Drill0.8mm -> Connector_PinHeader_2.54mm:PinHeader_1x02_P2.54mm_Vertical
- JP4: renamed from JP1; footprint TestPoint:TestPoint_2Pads_Pitch2.54mm_Drill0.8mm -> Connector_PinHeader_2.54mm:PinHeader_1x02_P2.54mm_Vertical
- JP5: renamed from JP4; footprint TestPoint:TestPoint_2Pads_Pitch2.54mm_Drill0.8mm -> Connector_PinHeader_2.54mm:PinHeader_1x02_P2.54mm_Vertical
- JP6: renamed from JP8; footprint TestPoint:TestPoint_2Pads_Pitch2.54mm_Drill0.8mm -> Connector_PinHeader_2.54mm:PinHeader_1x02_P2.54mm_Vertical
- JP7: renamed from JP6; footprint TestPoint:TestPoint_2Pads_Pitch2.54mm_Drill0.8mm -> Connector_PinHeader_2.54mm:PinHeader_1x02_P2.54mm_Vertical
- JP8: renamed from JP3; footprint TestPoint:TestPoint_2Pads_Pitch2.54mm_Drill0.8mm -> Connector_PinHeader_2.54mm:PinHeader_1x02_P2.54mm_Vertical
- JP9: renamed from JP10; footprint TestPoint:TestPoint_2Pads_Pitch2.54mm_Drill0.8mm -> Connector_PinHeader_2.54mm:PinHeader_1x02_P2.54mm_Vertical
- renumbered C5 to C40, C1 to C41, C33 to C42, C34 to C43, C36 to C44, C35 to C45, C37 to C46, C38 to C47, C40 to C48, C43 to C49, C39 to C50, C41 to C51, C42 to C52, D11 to D7, D14 to D8, D17 to D9, R19 to R28, R1 to R29, R17 to R30, R18 to R31, R20 to R32, U1 to U8
Connections:
- net VBAT renamed BATT
- net VRF renamed +VRF

Commit message: break out RF part to separate schema, update BOM
Parts:
- added J10: EXT 5V, Connector_PinHeader_2.54mm:PinHeader_1x02_P2.54mm_Vertical, symbol Connector_Generic:Conn_01x02
- added J11: EXT VRF, Connector_PinHeader_2.54mm:PinHeader_1x02_P2.54mm_Vertical, symbol Connector_Generic:Conn_01x02
- added J12: EXT 3V3, Connector_PinHeader_2.54mm:PinHeader_1x02_P2.54mm_Vertical, symbol Connector_Generic:Conn_01x02
- added J9: EXT VBAT, Connector_PinHeader_2.54mm:PinHeader_1x02_P2.54mm_Vertical, symbol Connector_Generic:Conn_01x02
- C16: renamed from C40; Part Number GRM033R61E104KE14J -> GRM155R61E104KA87D
- C17: renamed from C41; footprint Capacitor_SMD:C_0603_1608Metric_Pad1.08x0.95mm_HandSolder -> Capacitor_SMD:C_0805_2012Metric_Pad1.18x1.45mm_HandSolder; Part Number GRM21BR61H106KE43K -> GRM21BR61H106KE43L
- C20: renamed from C44; Part Number GRM033R61E104KE14J -> GRM155R61E104KA87D
- C21: renamed from C45; footprint Capacitor_SMD:C_0603_1608Metric_Pad1.08x0.95mm_HandSolder -> Capacitor_SMD:C_0805_2012Metric_Pad1.18x1.45mm_HandSolder; Part Number GRM21BR61H106KE43K -> GRM21BR61H106KE43L
- C24: renamed from C48; Part Number GRM033R61E104KE14J -> GRM155R61E104KA87D
- C25: renamed from C49; Manufactorer Murata -> Samsung; Part Number GRM033R61E104KE14J -> CL10C101JB8NNNC; Tolerance 10% -> 5%; Voltage 25 -> 50
- C26: renamed from C50; footprint Capacitor_SMD:C_0603_1608Metric_Pad1.08x0.95mm_HandSolder -> Capacitor_SMD:C_0805_2012Metric_Pad1.18x1.45mm_HandSolder; Part Number GRM21BR61H106KE43K -> GRM21BR61H106KE43L
- D7, D8: value GREEN V4 -> GREEN
- D9: value GREEN V3 -> GREEN
- L4: renamed from L7; Part Number DFE322512F-3R3M=P2 -> DFE322520FD-4R7M=P2
- R23: renamed from R28; Manufactorer (none) -> YAGEO; Part Number (none) -> RT0603BRD07165KL; Tolerance (none) -> 0.1%
- R24: renamed from R29; value 1k5 -> 1K5; Part Number RC0201FR-071K2L -> RC0603FR-071K5L
- R25: renamed from R30; Part Number RC0201FR-071K2L -> RC0603FR-071K2L
- R26: renamed from R31; Part Number RC0201FR-07680RL -> RC0603FR-07680RL
- R27: renamed from R32; Manufactorer (none) -> YAGEO; Part Number (none) -> RT0603BRD0733KL; Tolerance (none) -> 0.1%
- U5: renamed from U10; Part Number AP63203WU-7 -> AP63200WU-7; Voltage 3 -> variable
- renumbered C42 to C18, C43 to C19, C46 to C22, C47 to C23, C51 to C27, C52 to C28, L5 to L2, L6 to L3, U8 to U3, U9 to U4
Connections:
- net +3V3: now also J12.2 (Pin_2)
- net +5V: now also J10.2 (Pin_2)
- net +VBAT: now also J9.2 (Pin_2)
- net +VRF: now also J11.2 (Pin_2)
- net GND: now also J10.1 (Pin_1), J11.1 (Pin_1), J12.1 (Pin_1), J9.1 (Pin_1)
Other:
- note added: "External Power Inputs/Outputs"

Commit message: automatic schematic and pcb valiadation and cleanup
Parts:
- renumbered C16 to C51, C17 to C52, C18 to C53, C19 to C54, C20 to C55, C21 to C56, C22 to C57, C23 to C58, C24 to C59, C25 to C60, C26 to C61, C27 to C62, C28 to C63, D8 to D10, D9 to D11, D7 to D9, J9 to J11, J10 to J12, J11 to J13, J12 to J14, L2 to L1, L3 to L2, L4 to L3, R23 to R36, R24 to R37, R25 to R38, R26 to R39, R27 to R40, U3 to U10, U4 to U11, U5 to U12
