File: uart-can.kicad_sch (KiCad schematic)
At the start: 23 parts, among them J12 MS UART0, J13 MS Prog/Debug, J14 MS UART1, SW1 204-211ST, U11 MSPM0G3107SDGS20R, U12 TJA1051TK-3

Commit message: break out RF part to separate schema, update BOM
Parts:
- removed SW1: 204-211ST, Project:SW4_204-211ST_CTS, symbol Project:204-211ST
- added D10, D11: ORANGE, LED_SMD:LED_0603_1608Metric_Pad1.05x0.95mm_HandSolder, symbol Device:LED
- added R39, R40: 680, Resistor_SMD:R_0603_1608Metric_Pad0.98x0.95mm_HandSolder, symbol Device:R
- added S1: JS202011JCQN, Project:SW_JS202011JCQN, symbol Project:JS202011JCQN
- C29: renamed from C53; footprint Capacitor_SMD:C_0402_1005Metric_Pad0.74x0.62mm_HandSolder -> Capacitor_SMD:C_0603_1608Metric_Pad1.08x0.95mm_HandSolder; Manufactorer (none) -> Murata; Part Number (none) -> GRM21BR61E106KA73L; Tolerance (none) -> 10%; Voltage (none) -> 25
- C30: renamed from C54; Manufactorer (none) -> Murata; Part Number (none) -> GRM155R61E104KA87D; Tolerance (none) -> 10%; Voltage (none) -> 25
- C31: renamed from C55; Manufactorer (none) -> Samsung; Part Number (none) -> CL10A474KA8NNNC; Tolerance (none) -> 10%; Voltage (none) -> 25
- C32: renamed from C56; Manufactorer (none) -> Murata; Part Number (none) -> GRT1885C1E103JA02J; Tolerance (none) -> 5%; Voltage (none) -> 25
- C33: renamed from C57; Manufactorer (none) -> Murata; Part Number (none) -> GRM21BR61E106KA73L; Tolerance (none) -> 10%; Voltage (none) -> 25
- C34: renamed from C58; Manufactorer (none) -> Murata; Part Number (none) -> GRM155R61E104KA87D; Tolerance (none) -> 10%; Voltage (none) -> 25
- C35: renamed from C59; Manufactorer (none) -> Murata; Part Number (none) -> GRM21BR61E106KA73L; Tolerance (none) -> 10%; Voltage (none) -> 25
- C36: renamed from C60; Manufactorer (none) -> Murata; Part Number (none) -> GRM155R61E104KA87D; Tolerance (none) -> 10%; Voltage (none) -> 25
- C37: renamed from C61; Manufactorer (none) -> Samsung; Part Number (none) -> CL10C101JB8NNNC; Tolerance (none) -> 5%; Voltage (none) -> 50
- C38: renamed from C63; Manufactorer (none) -> Murata; Part Number (none) -> GRM1885C1H472JA01D; Tolerance (none) -> 5%; Voltage (none) -> 50
- C39: renamed from C62; Manufactorer (none) -> Samsung; Part Number (none) -> CL10C101JB8NNNC; Tolerance (none) -> 5%; Voltage (none) -> 50
- R28: renamed from R33; value 47k -> 47K; Manufactorer (none) -> YAGEO; Part Number (none) -> RT0603BRD0747KL; Tolerance (none) -> 1%
- R29: renamed from R34; value 100k -> 100K; Manufactorer (none) -> YAGEO; Part Number (none) -> RT0603BRD07100KL; Tolerance (none) -> 1%
- R30: renamed from R35; value 47k -> 47K; Manufactorer (none) -> YAGEO; Part Number (none) -> RT0603BRD0747KL; Tolerance (none) -> 1%
- R31: renamed from R37; Manufactorer (none) -> YAGEO; Part Number (none) -> RT0603BRD0720KL; Tolerance (none) -> 0.1%
- R32: renamed from R38; Manufactorer (none) -> YAGEO; Part Number (none) -> RT0603BRD060R4L; Tolerance (none) -> 1%
- R33: renamed from R39; Manufactorer (none) -> YAGEO; Part Number (none) -> RT0603BRD060R4L; Tolerance (none) -> 1%
- renumbered J12 to J13, J13 to J14, J14 to J15, U11 to U6, U12 to U7
Connections:
- net CAN_H: now also S1.5
- net CAN_L: now also S1.1
- net GND: now also R39.2, R40.2
- net MS_LED1: now reaches U6.8 (PA5_HFXIN_FCC_IN)
- net MS_LED1: now also D10.2 (A)
- net MS_LED2: now reaches U6.9 (PA6_HFCLK_IN_HFXOUT)
- net MS_LED2: now also D11.2 (A)
- net at R33.2: now also S1.2
- net at R32.2: now also S1.6
- new net: D11.1 (K), R40.1
- new net: D10.1 (K), R39.1
- no-connect marks 3 -> 1
Other:
- moved on the sheet: C37, C38, C39, R32, R33

Commit message: automatic schematic and pcb valiadation and cleanup
Parts:
- renumbered C29 to C40, C30 to C41, C31 to C42, C32 to C43, C33 to C44, C34 to C45, C35 to C46, C36 to C47, C37 to C48, C38 to C49, C39 to C50, D10 to D7, D11 to D8, J15 to J10, J13 to J8, J14 to J9, R39 to R34, R40 to R35, U6 to U8, U7 to U9
Connections:
- no-connect marks 1 -> 3
Other:
- moved on the sheet: C48, C49, C50, D7, D8, R32, R33, R34, R35
