File: openlst-hw.kicad_sch (KiCad schematic)
At the start: 8 parts

Commit message: temporary branch for radio to pc104
Parts:
- removed R1, R2, R3, R4: 22, Resistor_SMD:R_0603_1608Metric_Pad0.98x0.95mm_HandSolder, symbol Device:R
Connections:
- no-connect marks 23 -> 18
Other:
- removed sheet Power Converters
- removed sheet UART-CAN
- added sheet CAN Bridge (can_bridge.kicad_sch)
- sheet INTERBOARD_CONNECTOR2 ports: added *ATTENTION, *AVI_RST, *COMM1_RST, *COMM2_RST, *EPS_RST, *SCI_RST, BATT_1, BATT_2; removed 2V8_1, AVI_RESET, EPS_RESET, SCI_RST, UART_A_RXI, UART_A_TXO, UART_B_CTS, UART_B_RTS, UART_B_RXI, UART_B_TXO
- sheet MCU ports: added 3V3, GND, LST_RESET, LST_RX_MODE, LST_TX_MODE, PA_VAPC, RF_BYP, RF_EN, RF_N, RF_P, UART0_CTS, UART0_RTS, UART0_RX, UART0_TX, VRF; removed none
- sheet RF ports: added 3V3, GND, LST_RX_MODE, LST_TX_MODE, PA_VAPC, RF_BYP, RF_EN, RF_N, RF_P, VRF; removed none
- note removed: "Redundant in CubeSat all pwer from power board"
- note removed: "Relative to Avionics MCU"

Commit message: use Common libraries, replace TI MCU with STM32 for CAN bridge
Parts:
- H1, H2, H3, H4: footprint Project:MountingHole_4.3mm_M4_Pad_Via_Custom -> Common:MountingHole_4.3mm_M4_Pad_Via_Custom
Other:
- sheet MCU ports: added UART1_CTS, UART1_RTS, UART1_RX, UART1_TX; removed UART0_CTS, UART0_RTS, UART0_RX, UART0_TX
Changed lines of the file:
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@@
 	(hierarchical_label "3V3_BRIDGE"
 		(shape bidirectional)
-		(at 45.72 79.375 180)
+		(at 45.72 81.915 180)
 		(fields_autoplaced yes)
 		(effects
@@
 	(hierarchical_label "3V3_CAN"
 		(shape bidirectional)
-		(at 45.72 81.915 180)
+		(at 45.72 79.375 180)
 		(fields_autoplaced yes)
 		(effects
@@
 		(on_board yes)
 		(dnp no)
-		(property "Reference" "#PWR05"
+		(property "Reference" "#PWR01"
 			(at 140.97 196.85 0)
 			(effects
@@
 			(project ""
 				(path "/a863a5ec-a5d4-4f54-be53-e8c01d5e3ac4"
-					(reference "#PWR05")
+					(reference "#PWR01")
 					(unit 1)
 				)
@@
 			)
 		)
-		(property "Footprint" "Project:MountingHole_4.3mm_M4_Pad_Via_Custom"
+		(property "Footprint" "Common:MountingHole_4.3mm_M4_Pad_Via_Custom"
 			(at 151.13 171.45 0)
 			(effects
@@
 			)
 		)
-		(property "Footprint" "Project:MountingHole_4.3mm_M4_Pad_Via_Custom"
+		(property "Footprint" "Common:MountingHole_4.3mm_M4_Pad_Via_Custom"
 			(at 151.13 176.53 0)
 			(effects
@@
 			)
 		)
-		(property "Footprint" "Project:MountingHole_4.3mm_M4_Pad_Via_Custom"
+		(property "Footprint" "Common:MountingHole_4.3mm_M4_Pad_Via_Custom"
 			(at 151.13 181.61 0)
 			(effects
@@
 			)
 		)
-		(property "Footprint" "Project:MountingHole_4.3mm_M4_Pad_Via_Custom"
+		(property "Footprint" "Common:MountingHole_4.3mm_M4_Pad_Via_Custom"
 			(at 151.13 186.69 0)
 			(effects
@@
 		(dnp no)
 		(fields_autoplaced yes)
-		(property "Reference" "#FLG03"
+		(property "Reference" "#FLG02"
 			(at 109.855 106.68 0)
 			(effects
@@
 			(project "openlst-hw"
 				(path "/a863a5ec-a5d4-4f54-be53-e8c01d5e3ac4"
-					(reference "#FLG03")
+					(reference "#FLG02")
 					(unit 1)
 				)
@@
 		(dnp no)
 		(fields_autoplaced yes)
-		(property "Reference" "#FLG04"
+		(property "Reference" "#FLG03"
 			(at 132.715 106.68 0)
 			(effects
@@
 			(project "openlst-hw"
 				(path "/a863a5ec-a5d4-4f54-be53-e8c01d5e3ac4"
-					(reference "#FLG04")
+					(reference "#FLG03")
 					(unit 1)
 				)
@@
 		(dnp no)
 		(fields_autoplaced yes)
-		(property "Reference" "#FLG05"
+		(property "Reference" "#FLG04"
 			(at 151.13 106.68 0)
 			(effects
@@
 			(project "openlst-hw"
 				(path "/a863a5ec-a5d4-4f54-be53-e8c01d5e3ac4"
-					(reference "#FLG05")
+					(reference "#FLG04")
 					(unit 1)
 				)
@@
 		(dnp no)
 		(fields_autoplaced yes)
-		(property "Reference" "#FLG02"
+		(property "Reference" "#FLG01"
 			(at 86.36 106.68 0)
 			(effects
@@
 			(project ""
 				(path "/a863a5ec-a5d4-4f54-be53-e8c01d5e3ac4"
-					(reference "#FLG02")
+					(reference "#FLG01")
 					(unit 1)
 				)
@@
 			)
 		)
-		(pin "UART0_CTS" output
+		(pin "UART1_CTS" output
 			(at 154.305 59.69 180)
 			(effects
@@
 			)
 		)
-		(pin "UART0_RX" input
+		(pin "UART1_RX" input
 			(at 154.305 49.53 180)
 			(effects
@@
 			)
 		)
-		(pin "UART0_RTS" input
+		(pin "UART1_RTS" input
 			(at 154.305 57.15 180)
 			(effects
@@
 			)
 		)
-		(pin "UART0_TX" output
+		(pin "UART1_TX" output
 			(at 154.305 46.99 180)
 			(effects
